Commit message: update urdfs

File: Agents/models/talos_description_no_deps/urdf/talos_full_v2.urdf (robot description, URDF)
Before this commit: robot talos, 60 links, 59 joints
Links:
- link arm_left_1_link: geometry collision mesh filename=models/talos_description_no_deps/meshes/arm/arm_1_collision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 scale=1 1 1; visual mesh filename=models/talos_description_no_deps/meshes/arm/arm_1.STL scale=1 1 1
- link arm_left_2_link: geometry collision mesh filename=models/talos_description_no_deps/meshes/arm/arm_2_collision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 scale=1 1 1; visual mesh filename=models/talos_description_no_deps/meshes/arm/arm_2.STL scale=1 1 1
- link arm_left_3_link: geometry collision mesh filename=models/talos_description_no_deps/meshes/arm/arm_3_collision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 scale=1 1 1; visual mesh filename=models/talos_description_no_deps/meshes/arm/arm_3.STL scale=1 1 1
- link arm_left_4_link: geometry collision mesh filename=models/talos_description_no_deps/meshes/arm/arm_4_collision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 scale=1 1 1; visual mesh filename=models/talos_description_no_deps/meshes/arm/arm_4.STL scale=1 1 1
- link arm_left_5_link: geometry collision mesh filename=models/talos_description_no_deps/meshes/arm/arm_5_collision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 scale=1 1 1; visual mesh filename=models/talos_description_no_deps/meshes/arm/arm_5.STL scale=1 1 1
- link arm_left_6_link: geometry collision mesh filename=models/talos_description_no_deps/meshes/arm/arm_6_collision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 scale=1 1 1; visual mesh filename=models/talos_description_no_deps/meshes/arm/arm_6.STL scale=1 1 1
- link arm_left_7_link: geometry collision mesh filename=models/talos_description_no_deps/meshes/arm/arm_7_collision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 scale=1 1 1; visual mesh filename=models/talos_description_no_deps/meshes/arm/arm_7.STL scale=1 1 1
- link arm_right_1_link: geometry collision mesh filename=models/talos_description_no_deps/meshes/arm/arm_1_collision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 scale=1 -1 1; visual mesh filename=models/talos_description_no_deps/meshes/arm/arm_1.STL scale=1 -1 1
- link arm_right_2_link: geometry collision mesh filename=models/talos_description_no_deps/meshes/arm/arm_2_collision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 scale=1 -1 1; visual mesh filename=models/talos_description_no_deps/meshes/arm/arm_2.STL scale=1 -1 1
- link arm_right_3_link: geometry collision mesh filename=models/talos_description_no_deps/meshes/arm/arm_3_collision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 scale=1 -1 1; visual mesh filename=models/talos_description_no_deps/meshes/arm/arm_3.STL scale=1 -1 1
- link arm_right_4_link: geometry collision mesh filename=models/talos_description_no_deps/meshes/arm/arm_4_collision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 scale=1 -1 1; visual mesh filename=models/talos_description_no_deps/meshes/arm/arm_4.STL scale=1 -1 1
- link arm_right_5_link: geometry collision mesh filename=models/talos_description_no_deps/meshes/arm/arm_5_collision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 scale=1 -1 1; visual mesh filename=models/talos_description_no_deps/meshes/arm/arm_5.STL scale=1 -1 1
- link arm_right_6_link: geometry collision mesh filename=models/talos_description_no_deps/meshes/arm/arm_6_collision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 scale=1 -1 1; visual mesh filename=models/talos_description_no_deps/meshes/arm/arm_6.STL scale=1 -1 1
- link arm_right_7_link: geometry collision mesh filename=models/talos_description_no_deps/meshes/arm/arm_7_collision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 scale=1 -1 1; visual mesh filename=models/talos_description_no_deps/meshes/arm/arm_7.STL scale=1 -1 1
- link base_link: geometry collision mesh filename=models/talos_description_no_deps/meshes/torso/base_link_col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 scale=1 1 1; visual mesh filename=models/talos_description_no_deps/meshes/torso/base_link.STL scale=1 1 1
- link gripper_left_base_link: geometry collision mesh filename=models/talos_description_no_deps/meshes/gripper/base_link_c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 scale=1 1 1; visual mesh filename=models/talos_description_no_deps/meshes/gripper/base_link.S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 scale=1 1 1
- link gripper_left_fingertip_1_link: geometry collision mesh filename=models/talos_description_no_deps/meshes/gripper/fingertip_c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 scale=1 1 1; visual mesh filename=models/talos_description_no_deps/meshes/gripper/fingertip.S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 scale=1 1 1
- link gripper_left_fingertip_2_link: geometry collision mesh filename=models/talos_description_no_deps/meshes/gripper/fingertip_c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 scale=1 1 1; visual mesh filename=models/talos_description_no_deps/meshes/gripper/fingertip.S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 scale=1 1 1
- link gripper_left_fingertip_3_link: geometry collision mesh filename=models/talos_description_no_deps/meshes/gripper/fingertip_c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 scale=1 1 1; visual mesh filename=models/talos_description_no_deps/meshes/gripper/fingertip.S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 scale=1 1 1
- link gripper_left_inner_double_link: geometry collision mesh filename=models/talos_description_no_deps/meshes/gripper/inner_doubl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 scale=1 1 1; visual mesh filename=models/talos_description_no_deps/meshes/gripper/inner_doubl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 scale=1 1 1
- link gripper_left_inner_single_link: geometry collision mesh filename=models/talos_description_no_deps/meshes/gripper/inner_singl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 scale=1 1 1; visual mesh filename=models/talos_description_no_deps/meshes/gripper/inner_singl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 scale=1 1 1
- link gripper_left_motor_double_link: geometry collision mesh filename=models/talos_description_no_deps/meshes/gripper/gripper_mot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 scale=1 1 1; visual mesh filename=models/talos_description_no_deps/meshes/gripper/gripper_mot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 scale=1 1 1
- link gripper_left_motor_single_link: geometry collision mesh filename=models/talos_description_no_deps/meshes/gripper/gripper_mot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 scale=1 1 1; visual mesh filename=models/talos_description_no_deps/meshes/gripper/gripper_mot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 scale=1 1 1
- link gripper_right_base_link: geometry collision mesh filename=models/talos_description_no_deps/meshes/gripper/base_link_c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 scale=1 1 1; visual mesh filename=models/talos_description_no_deps/meshes/gripper/base_link.S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 scale=1 1 1
- link gripper_right_fingertip_1_link: geometry collision mesh filename=models/talos_description_no_deps/meshes/gripper/fingertip_c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 scale=1 1 1; visual mesh filename=models/talos_description_no_deps/meshes/gripper/fingertip.S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 scale=1 1 1
- link gripper_right_fingertip_2_link: geometry collision mesh filename=models/talos_description_no_deps/meshes/gripper/fingertip_c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 scale=1 1 1; visual mesh filename=models/talos_description_no_deps/meshes/gripper/fingertip.S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 scale=1 1 1
- link gripper_right_fingertip_3_link: geometry collision mesh filename=models/talos_description_no_deps/meshes/gripper/fingertip_c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 scale=1 1 1; visual mesh filename=models/talos_description_no_deps/meshes/gripper/fingertip.S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 scale=1 1 1
- link gripper_right_inner_double_link: geometry collision mesh filename=models/talos_description_no_deps/meshes/gripper/inner_doubl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 scale=1 1 1; visual mesh filename=models/talos_description_no_deps/meshes/gripper/inner_doubl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 scale=1 1 1
- link gripper_right_inner_single_link: geometry collision mesh filename=models/talos_description_no_deps/meshes/gripper/inner_singl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 scale=1 1 1; visual mesh filename=models/talos_description_no_deps/meshes/gripper/inner_singl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 scale=1 1 1
- link gripper_right_motor_double_link: geometry collision mesh filename=models/talos_description_no_deps/meshes/gripper/gripper_mot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 scale=1 1 1; visual mesh filename=models/talos_description_no_deps/meshes/gripper/gripper_mot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 scale=1 1 1
- link gripper_right_motor_single_link: geometry collision mesh filename=models/talos_description_no_deps/meshes/gripper/gripper_mot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 scale=1 1 1; visual mesh filename=models/talos_description_no_deps/meshes/gripper/gripper_mot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 scale=1 1 1
- link head_1_link: geometry collision mesh filename=models/talos_description_no_deps/meshes/head/head_1_collisi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 scale=1 1 1; visual mesh filename=models/talos_description_no_deps/meshes/head/head_1.stl scale=1 1 1
- link head_2_link: geometry collision mesh filename=models/talos_description_no_deps/meshes/head/head_2_collisi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 scale=1 1 1; visual mesh filename=models/talos_description_no_deps/meshes/head/head_2.stl scale=1 1 1
- link leg_left_1_link: geometry collision mesh filename=models/talos_description_no_deps/meshes/v2/hip_z_collision.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 scale=1 1 1; visual mesh filename=models/talos_description_no_deps/meshes/v2/hip_z_lo_res.stl scale=1 1 1
- link leg_left_2_link: geometry collision mesh filename=models/talos_description_no_deps/meshes/v2/hip_x_collision.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 scale=1 1 1; visual mesh filename=models/talos_description_no_deps/meshes/v2/hip_x_lo_res.stl scale=1 1 1
- link leg_left_3_link: geometry collision mesh filename=models/talos_description_no_deps/meshes/v2/hip_y_collision.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 scale=1 1 1; visual mesh filename=models/talos_description_no_deps/meshes/v2/hip_y_lo_res.stl scale=1 1 1
- link leg_left_4_link: geometry collision mesh filename=models/talos_description_no_deps/meshes/v2/knee_collision.s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 scale=1 1 1; visual mesh filename=models/talos_description_no_deps/meshes/v2/knee_lo_res.stl scale=1 1 1
- link leg_left_5_link: geometry collision mesh filename=models/talos_description_no_deps/meshes/v2/ankle_Y_collisio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 scale=1 1 1; visual mesh filename=models/talos_description_no_deps/meshes/v2/ankle_Y_lo_res.s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 scale=1 1 1
- link leg_left_6_link: geometry collision box size=0.21 0.13 0.02; visual mesh filename=models/talos_description_no_deps/meshes/v2/ankle_X_lo_res.s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 scale=1 1 1
- link leg_right_1_link: geometry collision mesh filename=models/talos_description_no_deps/meshes/v2/hip_z_collision.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 scale=1 -1 1; visual mesh filename=models/talos_description_no_deps/meshes/v2/hip_z_lo_res.stl scale=1 -1 1
- link leg_right_2_link: geometry collision mesh filename=models/talos_description_no_deps/meshes/v2/hip_x_collision.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 scale=1 -1 1; visual mesh filename=models/talos_description_no_deps/meshes/v2/hip_x_lo_res.stl scale=1 -1 1
- link leg_right_3_link: geometry collision mesh filename=models/talos_description_no_deps/meshes/v2/hip_y_collision.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 scale=1 -1 1; visual mesh filename=models/talos_description_no_deps/meshes/v2/hip_y_lo_res.stl scale=1 -1 1
- link leg_right_4_link: geometry collision mesh filename=models/talos_description_no_deps/meshes/v2/knee_collision.s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 scale=1 -1 1; visual mesh filename=models/talos_description_no_deps/meshes/v2/knee_lo_res.stl scale=1 -1 1
- link leg_right_5_link: geometry collision mesh filename=models/talos_description_no_deps/meshes/v2/ankle_Y_collisio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 scale=1 -1 1; visual mesh filename=models/talos_description_no_deps/meshes/v2/ankle_Y_lo_res.s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 scale=1 -1 1
- link leg_right_6_link: geometry collision box size=0.21 0.13 0.02; visual mesh filename=models/talos_description_no_deps/meshes/v2/ankle_X_lo_res.s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 scale=1 -1 1
- link rgbd_link: geometry collision box size=0.04 0.185 0.03; visual mesh filename=models/talos_description_no_deps/meshes/sensors/orbbec/orbb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
- link torso_1_link: geometry collision mesh filename=models/talos_description_no_deps/meshes/torso/torso_1.STL scale=1 1 1; visual mesh filename=models/talos_description_no_deps/meshes/torso/torso_1.STL scale=1 1 1
- link torso_2_link: geometry collision mesh filename=models/talos_description_no_deps/meshes/torso/torso_2_colli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 scale=1 1 1; visual mesh filename=models/talos_description_no_deps/meshes/torso/torso_2.STL scale=1 1 1
